File: Eagle/USBpassthru/passthru.sch (EAGLE design)
At the start: 4 parts

Commit message: Add PIN HEADER package and connections
Parts:
- added CHG: (no value), pinhead:PINHD-1X1
Connections:
- net +5V: now also CHG.1
Changed lines of the file:
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@@
 <part name="+" library="pinhead" library_urn="urn:adsk.eagle:library:325" deviceset="PINHD-1X2" device="" package3d_urn="urn:adsk.eagle:package:22435/2" value="plug"/>
 <part name="GND1" library="supply1" deviceset="GND" device=""/>
+<part name="CHG" library="pinhead" library_urn="urn:adsk.eagle:library:325" deviceset="PINHD-1X1" device="" package3d_urn="urn:adsk.eagle:package:22485/2"/>
 </parts>
 <sheets>
@@
 <attribute name="VALUE" x="43.18" y="30.48" size="1.778" layer="96"/>
 </instance>
+<instance part="CHG" gate="G$1" x="73.66" y="48.26" smashed="yes">
+<attribute name="NAME" x="67.31" y="51.435" size="1.778" layer="95"/>
+<attribute name="VALUE" x="67.31" y="43.18" size="1.778" layer="96"/>
+</instance>
 </instances>
 <busses>
@@
 <pinref part="PMEG2005CT" gate="G$1" pin="A1"/>
 <wire x1="50.8" y1="55.88" x2="50.8" y2="58.42" width="0.1524" layer="91"/>
-<wire x1="50.8" y1="58.42" x2="76.2" y2="58.42" width="0.1524" layer="91"/>
+<wire x1="50.8" y1="58.42" x2="63.5" y2="58.42" width="0.1524" layer="91"/>
+<wire x1="63.5" y1="58.42" x2="76.2" y2="58.42" width="0.1524" layer="91"/>
 <wire x1="76.2" y1="58.42" x2="76.2" y2="55.88" width="0.1524" layer="91"/>
 <junction x="76.2" y="58.42"/>
+<pinref part="CHG" gate="G$1" pin="1"/>
+<wire x1="71.12" y1="48.26" x2="63.5" y2="48.26" width="0.1524" layer="91"/>
+<wire x1="63.5" y1="48.26" x2="63.5" y2="58.42" width="0.1524" layer="91"/>
+<junction x="63.5" y="58.42"/>
 </segment>
 </net>
